Commit message: fix cafe_table v1.0

File: src/lab4_pkg/src/cafe_table.xacro (robot description, xacro)
@@ -33,8 +33,8 @@
   </link>
   <joint name="cafe_table_fixed" type="fixed">
-  <origin rpy="0 0 0" xyz="1.0 0 -0.93"/>
-  <axis xyz="0 0 1"/>
-  <parent link="world"/>
-  <child link="cafe_table__link"/>
+    <origin rpy="0 0 0" xyz="1.0 0 -0.93"/>
+    <axis xyz="0 0 1"/>
+    <parent link="world"/>
+    <child link="cafe_table__link"/>
 </joint>
 </robot>
