Commit message: baxter folder modified

File: src/baxter/baxter/baxter_common/baxter_description/urdf/baxter.urdf.xacro (robot description, xacro)
@@ -1,15 +1,14 @@
-<?xml version="1.0" ?>
+<?xml version="1.0"?>
 <robot name="baxter" xmlns:xacro="http://www.ros.org/wiki/xacro">
-  <xacro:arg name="gazebo" default="true"/>
-  <xacro:arg name="pedestal" default="true"/>
-  <xacro:arg name="coffe_table" default="true"/>
+  <xacro:arg name="gazebo" default="false" />
+  <xacro:arg name="pedestal" default="true" />
   <!-- Baxter Base URDF -->
   <xacro:include filename="$(find baxter_description)/urdf/baxter_base/baxter_base.urdf.xacro">
-    <xacro:arg name="gazebo" value="${gazebo}"/>
+    <xacro:arg name="gazebo" value="${gazebo}" />
   </xacro:include>
   <!-- Baxter Pedestal -->
   <xacro:if value="$(arg pedestal)">
     <xacro:include filename="$(find baxter_description)/urdf/pedestal/pedestal.xacro">
-      <xacro:arg name="gazebo" value="${gazebo}"/>
+      <xacro:arg name="gazebo" value="${gazebo}" />
     </xacro:include>
   </xacro:if>
@@ -18,10 +17,10 @@
   <!-- Right End Effector -->
   <xacro:include filename="$(find baxter_description)/urdf/right_end_effector.urdf.xacro" />
-  <!-- Coffe Table -->
-  <xacro:include filename="$(find baxter_sim_examples)/models/cafe_table/cafe_table.xacro" />
   <!-- Kinect Sensor -->
   <xacro:if value="$(arg gazebo)">
     <xacro:include filename="$(find baxter_description)/urdf/depth_sensor.urdf.xacro" />
-    <sensor_kinect parent="base" location="1.0 -0.0125 2.0" orientation="0 1.57 0.0"/>
+    <sensor_kinect parent="base" location="1.0 -0.0125 2.0" orientation="0 1.57 0.0" />
   </xacro:if>
+  <!-- Coffe Table -->
+  <xacro:include filename="$(find baxter_sim_examples)/models/cafe_table/cafe_table.xacro" />
 </robot>

File: src/baxter/baxter/baxter_common/baxter_description/urdf/baxter_lab.urdf (robot description, URDF)
Before this commit: robot baxter, 57 links, 56 joints
Links:
- added link cafe_table__link, mass 0; collision box size=0.042 0.042 0.74; collision box size=0.56 0.56 0.04
Joints:
- added joint cafe_table_fixed: type fixed, parent world, child cafe_table__link, origin xyz=1.0 0 -0.93 rpy=0 0 0, axis 0 0 1

File: src/baxter/baxter/baxter_common/baxter_description/urdf/depth_sensor.urdf.xacro (robot description, xacro)
@@ -1,12 +1,12 @@
 <?xml version="1.0"?>
 <robot name="depth_sensor" xmlns:xacro="http://ros.org/wiki/xacro">
-  <xacro:include filename="$(find baxter_description)/urdf/kinect_sim.urdf.xacro"/>
+  <xacro:include filename="$(find baxter_description)/urdf/kinect_sim.urdf.xacro" />
   <xacro:macro name="sensor_kinect" params="parent location orientation">
     <joint name="camera_rgb_joint" type="fixed">
-      <origin xyz="${location}" rpy="${orientation}"/>
-      <parent link="${parent}"/>
+      <origin xyz="${location}" rpy="${orientation}" />
+      <parent link="${parent}" />
       <child link="camera_rgb_frame" />
     </joint>
-    <link name="camera_rgb_frame"/>
+    <link name="camera_rgb_frame" />
     <joint name="camera_rgb_optical_joint" type="fixed">
       <origin xyz="0 0 0" rpy="${-M_PI/2} 0 ${-M_PI/2}" />
@@ -14,34 +14,34 @@
       <child link="camera_rgb_optical_frame" />
     </joint>
-    <link name="camera_rgb_optical_frame"/>
+    <link name="camera_rgb_optical_frame" />
     <joint name="camera_joint" type="fixed">
-      <origin xyz="0 0 0" rpy="0 0 0"/> <!-- -0.031 -0.0125 -0.016 -->
-      <parent link="camera_rgb_frame"/>
-      <child link="camera_link"/>
+      <origin xyz="0 0 0" rpy="0 0 0" /> <!-- -0.031 -0.0125 -0.016 -->
+      <parent link="camera_rgb_frame" />
+      <child link="camera_link" />
     </joint>
-      <link name="camera_link">
+    <link name="camera_link">
       <visual>
-       <origin xyz="0 0 0" rpy="0 0 0"/>
+        <origin xyz="0 0 0" rpy="0 0 0" />
         <geometry>
-         <mesh filename="package://baxter_description/meshes/kinect.dae"/>
+          <mesh filename="package://baxter_description/meshes/kinect.dae" />
         </geometry>
       </visual>
-        <collision>
-        <origin xyz="0.0 0.0 0.0" rpy="0 0 0"/>
-          <geometry>
-            <box size="0.07271 0.27794 0.073"/>
-          </geometry>
-        </collision>
+      <collision>
+        <origin xyz="0.0 0.0 0.0" rpy="0 0 0" />
+        <geometry>
+          <box size="0.07271 0.27794 0.073" />
+        </geometry>
+      </collision>
       <inertial>
         <mass value="0.564" />
         <origin xyz="0 0 0" />
         <inertia ixx="0.003881243" ixy="0.0" ixz="0.0"
-                 iyy="0.000498940" iyz="0.0"
-                 izz="0.003879257" />
+          iyy="0.000498940" iyz="0.0"
+          izz="0.003879257" />
       </inertial>
     </link>
-    <!-- The fixed joints & links below are usually published by static_transformers launched by the OpenNi launch
-         files. However, for Gazebo simulation we need them, so we add them here.
-         (Hence, don't publish them additionally!) -->
+    <!-- The fixed joints & links below are usually published by static_transformers launched by the
+    OpenNi launch files. However, for Gazebo simulation we need them, so we add them here and aren't
+    published by static_transformers!) -->
     <joint name="camera_depth_joint" type="fixed">
       <origin xyz="0 ${2 * 0.0125} 0" rpy="0 0 0" />
@@ -49,5 +49,5 @@
       <child link="camera_depth_frame" />
     </joint>
-    <link name="camera_depth_frame"/>
+    <link name="camera_depth_frame" />
     <joint name="camera_depth_optical_joint" type="fixed">
       <origin xyz="0 0 0" rpy="${-M_PI/2} 0 ${-M_PI/2}" />
@@ -55,7 +55,7 @@
       <child link="camera_depth_optical_frame" />
     </joint>
-    <link name="camera_depth_optical_frame"/>
+    <link name="camera_depth_optical_frame" />
     <!-- Kinect sensor for simulation -->
-    <kinect_camera/>
+    <kinect_camera />
   </xacro:macro>
 </robot>

File: src/baxter/baxter/baxter_common/baxter_description/urdf/kinect_sim.urdf.xacro (robot description, xacro)
@@ -22,5 +22,5 @@
           <cameraName>camera</cameraName>
           <alwaysOn>true</alwaysOn>
-          <updateRate>10</updateRate>
+          <updateRate>5</updateRate>
           <imageTopicName>rgb/image_raw</imageTopicName>
           <depthImageTopicName>depth/image_raw</depthImageTopicName>

File: src/baxter/baxter/baxter_common/baxter_description/urdf/left_end_effector.urdf.xacro (robot description, xacro)
@@ -1,13 +1,14 @@
-<?xml version="1.0" ?>
+<?xml version="1.0"?>
 <robot name="left_end_effector" xmlns:xacro="http://www.ros.org/wiki/xacro">
-  <xacro:include filename="$(find rethink_ee_description)/urdf/electric_gripper/rethink_electric_gripper.xacro" />
+  <xacro:include
+    filename="$(find rethink_ee_description)/urdf/electric_gripper/rethink_electric_gripper.xacro" />
   <xacro:rethink_electric_gripper side="left"
-                                  l_finger="extended_narrow"
-                                  l_finger_slot="2"
-                                  l_finger_tip="paddle_tip"
-                                  l_finger_grasp="inner"
-                                  r_finger="extended_narrow"
-                                  r_finger_slot="2"
-                                  r_finger_tip="paddle_tip"
-                                  r_finger_grasp="inner"/>
+    l_finger="extended_narrow"
+    l_finger_slot="2"
+    l_finger_tip="paddle_tip"
+    l_finger_grasp="inner"
+    r_finger="extended_narrow"
+    r_finger_slot="2"
+    r_finger_tip="paddle_tip"
+    r_finger_grasp="inner" />
 </robot>

File: src/baxter/baxter/baxter_common/baxter_description/urdf/right_end_effector.urdf.xacro (robot description, xacro)
@@ -1,13 +1,14 @@
-<?xml version="1.0" ?>
+<?xml version="1.0"?>
 <robot name="right_end_effector" xmlns:xacro="http://www.ros.org/wiki/xacro">
-  <xacro:include filename="$(find rethink_ee_description)/urdf/electric_gripper/rethink_electric_gripper.xacro" />
+  <xacro:include
+    filename="$(find rethink_ee_description)/urdf/electric_gripper/rethink_electric_gripper.xacro" />
   <xacro:rethink_electric_gripper side="right"
-                                  l_finger="extended_narrow"
-                                  l_finger_slot="2"
-                                  l_finger_tip="half_round_tip"
-                                  l_finger_grasp="inner"
-                                  r_finger="extended_narrow"
-                                  r_finger_slot="2"
-                                  r_finger_tip="half_round_tip"
-                                  r_finger_grasp="inner"/>
+    l_finger="extended_narrow"
+    l_finger_slot="2"
+    l_finger_tip="half_round_tip"
+    l_finger_grasp="inner"
+    r_finger="extended_narrow"
+    r_finger_slot="2"
+    r_finger_tip="half_round_tip"
+    r_finger_grasp="inner" />
 </robot>
