Commit message: lab5 and chess hot fixes

File: install/share/baxter_description/urdf/baxter.urdf.xacro (robot description, xacro)
@@ -1,14 +1,14 @@
-<?xml version="1.0" ?>
+<?xml version="1.0"?>
 <robot name="baxter" xmlns:xacro="http://www.ros.org/wiki/xacro">
-  <xacro:arg name="gazebo" default="false"/>
-  <xacro:arg name="pedestal" default="true"/>
+  <xacro:arg name="gazebo" default="false" />
+  <xacro:arg name="pedestal" default="true" />
   <!-- Baxter Base URDF -->
   <xacro:include filename="$(find baxter_description)/urdf/baxter_base/baxter_base.urdf.xacro">
-    <xacro:arg name="gazebo" value="${gazebo}"/>
+    <xacro:arg name="gazebo" value="${gazebo}" />
   </xacro:include>
   <!-- Baxter Pedestal -->
   <xacro:if value="$(arg pedestal)">
     <xacro:include filename="$(find baxter_description)/urdf/pedestal/pedestal.xacro">
-      <xacro:arg name="gazebo" value="${gazebo}"/>
+      <xacro:arg name="gazebo" value="${gazebo}" />
     </xacro:include>
   </xacro:if>
@@ -18,6 +18,8 @@
   <xacro:include filename="$(find baxter_description)/urdf/right_end_effector.urdf.xacro" />
   <!-- Kinect Sensor -->
-  <xacro:include filename="$(find baxter_description)/urdf/depth_sensor.urdf.xacro" />
-  <sensor_kinect parent="base" location="1.0 -0.0125 2.0" orientation="0 1.57 0.0"/>
+  <xacro:if value="$(arg gazebo)">
+    <xacro:include filename="$(find baxter_description)/urdf/depth_sensor.urdf.xacro" />
+    <sensor_kinect parent="base" location="1.0 -0.0125 2.0" orientation="0 1.57 0.0" />
+  </xacro:if>
   <!-- Coffe Table -->
   <xacro:include filename="$(find baxter_sim_examples)/models/cafe_table/cafe_table.xacro" />

File: install/share/baxter_description/urdf/depth_sensor.urdf.xacro (robot description, xacro)
@@ -1,12 +1,12 @@
 <?xml version="1.0"?>
 <robot name="depth_sensor" xmlns:xacro="http://ros.org/wiki/xacro">
-  <xacro:include filename="$(find baxter_description)/urdf/kinect_sim.urdf.xacro"/>
+  <xacro:include filename="$(find baxter_description)/urdf/kinect_sim.urdf.xacro" />
   <xacro:macro name="sensor_kinect" params="parent location orientation">
     <joint name="camera_rgb_joint" type="fixed">
-      <origin xyz="${location}" rpy="${orientation}"/>
-      <parent link="${parent}"/>
+      <origin xyz="${location}" rpy="${orientation}" />
+      <parent link="${parent}" />
       <child link="camera_rgb_frame" />
     </joint>
-    <link name="camera_rgb_frame"/>
+    <link name="camera_rgb_frame" />
     <joint name="camera_rgb_optical_joint" type="fixed">
       <origin xyz="0 0 0" rpy="${-M_PI/2} 0 ${-M_PI/2}" />
@@ -14,32 +14,34 @@
       <child link="camera_rgb_optical_frame" />
     </joint>
-    <link name="camera_rgb_optical_frame"/>
+    <link name="camera_rgb_optical_frame" />
     <joint name="camera_joint" type="fixed">
-      <origin xyz="0 0 0" rpy="0 0 0"/> <!-- -0.031 -0.0125 -0.016 -->
-      <parent link="camera_rgb_frame"/>
-      <child link="camera_link"/>
+      <origin xyz="0 0 0" rpy="0 0 0" /> <!-- -0.031 -0.0125 -0.016 -->
+      <parent link="camera_rgb_frame" />
+      <child link="camera_link" />
     </joint>
-      <link name="camera_link">
+    <link name="camera_link">
       <visual>
-       <origin xyz="0 0 0" rpy="0 0 0"/>
+        <origin xyz="0 0 0" rpy="0 0 0" />
         <geometry>
-         <mesh filename="package://baxter_description/meshes/kinect.dae"/>
+          <mesh filename="package://baxter_description/meshes/kinect.dae" />
         </geometry>
       </visual>
-        <collision>
-        <origin xyz="0.0 0.0 0.0" rpy="0 0 0"/>
-          <geometry>
-            <box size="0.07271 0.27794 0.073"/>
-          </geometry>
-        </collision>
+      <collision>
+        <origin xyz="0.0 0.0 0.0" rpy="0 0 0" />
+        <geometry>
+          <box size="0.07271 0.27794 0.073" />
+        </geometry>
+      </collision>
       <inertial>
         <mass value="0.564" />
         <origin xyz="0 0 0" />
         <inertia ixx="0.003881243" ixy="0.0" ixz="0.0"
-                 iyy="0.000498940" iyz="0.0"
-                 izz="0.003879257" />
+          iyy="0.000498940" iyz="0.0"
+          izz="0.003879257" />
       </inertial>
     </link>
-    <!-- The fixed joints & links below are usually published by static_transformers launched by the OpenNi launch files. However, for Gazebo simulation we need them, so we add them here and aren't published by static_transformers!) -->
+    <!-- The fixed joints & links below are usually published by static_transformers launched by the
+    OpenNi launch files. However, for Gazebo simulation we need them, so we add them here and aren't
+    published by static_transformers!) -->
     <joint name="camera_depth_joint" type="fixed">
       <origin xyz="0 ${2 * 0.0125} 0" rpy="0 0 0" />
@@ -47,5 +49,5 @@
       <child link="camera_depth_frame" />
     </joint>
-    <link name="camera_depth_frame"/>
+    <link name="camera_depth_frame" />
     <joint name="camera_depth_optical_joint" type="fixed">
       <origin xyz="0 0 0" rpy="${-M_PI/2} 0 ${-M_PI/2}" />
@@ -53,7 +55,7 @@
       <child link="camera_depth_optical_frame" />
     </joint>
-    <link name="camera_depth_optical_frame"/>
+    <link name="camera_depth_optical_frame" />
     <!-- Kinect sensor for simulation -->
-    <kinect_camera/>
+    <kinect_camera />
   </xacro:macro>
 </robot>
