Commit message: lab4, 5 and chess adjusted for rebuild

File: rf_ws/src/lab4_pkg/src/cafe_table.xacro (robot description, xacro)
@@ -37,4 +37,4 @@
     <parent link="world"/>
     <child link="cafe_table__link"/>
-</joint>
+  </joint>
 </robot>

File: src/baxter/baxter/baxter_simulator/baxter_sim_examples/models/cafe_table/cafe_table.xacro (robot description, xacro)
@@ -33,5 +33,5 @@
   </link>
   <joint name="cafe_table_fixed" type="fixed">
-    <origin rpy="0 0 0" xyz="0.78 0.3 -0.93"/>
+    <origin rpy="0 0 0" xyz="1.0 0 -0.93"/>
     <axis xyz="0 0 1"/>
     <parent link="world"/>
